File: sap1-mk2/rega.kicad_sch (KiCad schematic)
At the start: 0 parts

Commit message: added A Register, B Register, Instruction Register, and Memory Address Register
Parts:
- added C12, C13, C14: 0.1μF, symbol Device:C_Small
- added D2, D3, D4, D5, D6, D7, D8, D9: RED, symbol Device:LED
- added R10, R11, R12, R13, R14, R15, R8, R9: 220, symbol Device:R
- added U7: 74LS245, symbol 74xx:74LS245
- added U8, U9: 74LS173, symbol 74xx:74LS173
Connections:
- new net: D8.1 (K), R14.1
- new net: D6.1 (K), R12.1
- new net: D9.1 (K), R15.1
- new net: D5.1 (K), R11.1
- new net: D3.1 (K), R9.1
- new net: D7.1 (K), R13.1
- new net: D2.1 (K), R8.1
- new net: D4.1 (K), R10.1
- new net +5V: C12.2, C13.2, C14.2, U7.1 (A->B), U7.20 (VCC), U8.16 (VCC), U9.16 (VCC)
- new net A_0: D9.2 (A), U7.9 (A7), U9.6 (Q3)
- new net A_1: D8.2 (A), U7.8 (A6), U9.5 (Q2)
- new net A_2: D7.2 (A), U7.7 (A5), U9.4 (Q1)
- new net A_3: D6.2 (A), U7.6 (A4), U9.3 (Q0)
- new net A_4: D5.2 (A), U7.5 (A3), U8.6 (Q3)
- new net A_5: D4.2 (A), U7.4 (A2), U8.5 (Q2)
- new net A_6: D3.2 (A), U7.3 (A1), U8.4 (Q1)
- new net A_7: D2.2 (A), U7.2 (A0), U8.3 (Q0)
- new net BUS_0: U7.11 (B7), U9.11 (D3)
- new net BUS_1: U7.12 (B6), U9.12 (D2)
- new net BUS_2: U7.13 (B5), U9.13 (D1)
- new net BUS_3: U7.14 (B4), U9.14 (D0)
- new net BUS_4: U7.15 (B3), U8.11 (D3)
- new net BUS_5: U7.16 (B2), U8.12 (D2)
- new net BUS_6: U7.17 (B1), U8.13 (D1)
- new net BUS_7: U7.18 (B0), U8.14 (D0)
- new net CLK: U8.7 (Cp), U9.7 (Cp)
- new net CLR: U8.15 (Mr), U9.15 (Mr)
- new net GND: C12.1, C13.1, C14.1, R10.2, R11.2, R12.2, R13.2, R14.2, R15.2, R8.2, R9.2, U7.10 (GND), U8.1 (Oe1), U8.2 (Oe2), U8.8 (GND), U9.1 (Oe1), U9.2 (Oe2), U9.8 (GND)
- new net ~{AI}: U8.10 (E2), U8.9 (E1), U9.10 (E2), U9.9 (E1)
- new net ~{AO}: U7.19 (CE)
Other:
- title: (none) -> A Register
