File: sap1-mk2/alu.kicad_sch (KiCad schematic)
At the start: 0 parts

Commit message: added ALU + some minor tweaks
Parts:
- added C23, C24, C25, C26, C27, C28, C29, C30: 0.1μF, symbol Device:C_Small
- added D32, D33: GREEN, symbol Device:LED
- added D34, D35, D36, D37, D38, D39, D40, D41: RED, symbol Device:LED
- added R38, R39, R40, R41, R42, R43, R44, R45, R46, R47: 220, symbol Device:R
- added U18: 74LS173, symbol 74xx:74LS173
- added U19: 74LS08, symbol 74xx:74LS08
- added U20: 74LS02, symbol 74xx:74LS02
- added U21: 74LS245, symbol 74xx:74LS245
- added U22, U23: 74LS283, symbol 74xx_IEEE:74LS283
- added U24, U25: 74LS86, symbol 74xx:74LS86
Connections:
- new net: U19.1, U20.1
- new net: U19.2, U20.4
- new net: U19.3, U19.4
- new net: U23.15 (B3), U25.11
- new net: D37.1 (K), R43.2
- new net: D37.2 (A), U20.6, U21.5 (A3), U22.4 (S1)
- new net: D35.1 (K), R41.2
- new net: D40.2 (A), U20.11, U21.8 (A6), U23.1 (S2)
- new net: D41.2 (A), U20.12, U21.9 (A7), U23.4 (S1)
- new net: U19.10, U20.13
- new net: U19.5, U19.8
- new net: U18.13 (D1), U19.6
- new net: U23.2 (B2), U25.3
- new net: D40.1 (K), R46.2
- new net: D39.1 (K), R45.2
- new net: D39.2 (A), U20.9, U21.7 (A5), U23.13 (S3)
- new net: D36.1 (K), R42.2
- new net: D32.1 (K), R39.1
- new net: D38.2 (A), U20.8, U21.6 (A4), U23.10 (S4)
- new net: U23.11 (B4), U25.8
- new net: C28.2, U23.16 (VCC)
- new net: U23.6 (B1), U25.6
- new net: C28.1, U23.8 (GND)
- new net: U22.7 (C0), U23.9 (C4)
- new net: U19.9, U20.10
- new net: D38.1 (K), R44.2
- new net: U22.11 (B4), U24.8
- new net: D34.1 (K), R40.2
- new net: U22.15 (B3), U24.11
- new net: D36.2 (A), U20.5, U21.4 (A2), U22.1 (S2)
- new net: C27.1, U22.8 (GND)
- new net: C27.2, U22.16 (VCC)
- new net: D33.1 (K), R38.1
- new net: D34.2 (A), U20.2, U21.2 (A0), U22.10 (S4)
- new net: D35.2 (A), U20.3, U21.3 (A1), U22.13 (S3)
- new net: U22.2 (B2), U24.3
- new net: U22.6 (B1), U24.6
- new net: U18.14 (D0), U22.9 (C4)
- new net: D41.1 (K), R47.2
- new net +5V: C23.1, C24.2, C25.2, C26.1, C29.2, C30.2, U18.16 (VCC), U19.14 (VCC), U20.14 (VCC), U21.1 (A->B), U21.20 (VCC), U24.14 (VCC), U25.14 (VCC)
- new net A_0: U23.5 (A1)
- new net A_1: U23.3 (A2)
- new net A_2: U23.14 (A3)
- new net A_3: U23.12 (A4)
- new net A_4: U22.5 (A1)
- new net A_5: U22.3 (A2)
- new net A_6: U22.14 (A3)
- new net A_7: U22.12 (A4)
- new net BUS_0: U21.11 (B7)
- new net BUS_1: U21.12 (B6)
- new net BUS_2: U21.13 (B5)
- new net BUS_3: U21.14 (B4)
- new net BUS_4: U21.15 (B3)
- new net BUS_5: U21.16 (B2)
- new net BUS_6: U21.17 (B1)
- new net BUS_7: U21.18 (B0)
- new net B_0: U25.4
- new net B_1: U25.1
- new net B_2: U25.12
- new net B_3: U25.9
- new net B_4: U24.4
- new net B_5: U24.1
- new net B_6: U24.12
- new net B_7: U24.9
- new net CF: D33.2 (A), U18.3 (Q0)
- new net CLK: U18.7 (Cp)
- new net CLR: U18.15 (Mr)
- new net GND: C23.2, C24.1, C25.1, C26.2, C29.1, C30.1, R38.2, R39.2, R40.1, R41.1, R42.1, R43.1, R44.1, R45.1, R46.1, R47.1, U18.1 (Oe1), U18.2 (Oe2), U18.8 (GND), U19.12, U19.13, U19.7 (GND), U20.7 (GND), U21.10 (GND), U24.7 (GND), U25.7 (GND)
- new net SU: U23.7 (C0), U24.10, U24.13, U24.2, U24.5, U25.10, U25.13, U25.2, U25.5
- new net ZF: D32.2 (A), U18.4 (Q1)
- new net ~{EO}: U21.19 (CE)
- new net ~{FI}: U18.10 (E2), U18.9 (E1)
- no-connect marks 0 -> 5
Other:
- title: (none) -> Arithmetic Logic Unit
