File: sap1-mk2/progcounter.kicad_sch (KiCad schematic)
At the start: 0 parts

Commit message: added program counter schematic
Parts:
- added C31, C32: 0.1μF, symbol Device:C_Small
- added D42, D43, D44, D45: GREEN, symbol Device:LED
- added R48, R49, R50, R51: 220, symbol Device:R
- added U26: 74LS245, symbol 74xx:74LS245
- added U27: 74LS161, symbol 74xx:74LS161
Connections:
- new net: D43.1 (K), R49.2
- new net: D42.2 (A), U26.14 (B4), U27.11 (Q3)
- new net: D43.2 (A), U26.13 (B5), U27.12 (Q2)
- new net: D44.2 (A), U26.12 (B6), U27.13 (Q1)
- new net: D45.2 (A), U26.11 (B7), U27.14 (Q0)
- new net: D44.1 (K), R50.2
- new net: D45.1 (K), R51.2
- new net: D42.1 (K), R48.2
- new net +5V: C31.1, C32.1, U26.20 (VCC), U27.16 (VCC)
- new net BUS_0: U26.9 (A7), U27.6 (D3)
- new net BUS_1: U26.8 (A6), U27.5 (D2)
- new net BUS_2: U26.7 (A5), U27.4 (D1)
- new net BUS_3: U26.6 (A4), U27.3 (D0)
- new net CE: U27.10 (CET), U27.7 (CEP)
- new net CLK: U27.2 (CP)
- new net GND: C31.2, C32.2, R48.1, R49.1, R50.1, R51.1, U26.1 (A->B), U26.10 (GND), U27.8 (GND)
- new net ~{CLR}: U27.1 (~{MR})
- new net ~{CO}: U26.19 (CE)
- new net ~{J}: U27.9 (~{PE})
- no-connect marks 0 -> 9
