File: sap1_mk2/controllogic.kicad_sch (KiCad schematic)
At the start: 0 parts

Commit message: finished schematics rev 1.0 // added Control Logic
Parts:
- added C48, C49, C50, C51, C52, C53: 0.1μF, symbol Device:C_Small
- added D54, D55, D56: RED, symbol Device:LED
- added D57, D58, D59, D60, D61: GREEN, symbol Device:LED
- added D62, D63, D64, D65, D66, D67, D68, D69, D70, D71, D72, D73, D74, D75, D76, D77: BLUE, symbol Device:LED
- added R72, R73, R74, R75, R76, R77, R78, R79, R81, R82, R83, R84, R85, R86, R87, R88, R89, R90, R91, R92, R93, R94, R95, R96: 220, symbol Device:R
- added R80: 1K, symbol Device:R
- added SW8: Reset, symbol Switch:SW_Push
- added U45, U46: AT28C16, Package_DIP:DIP-24_W15.24mm, symbol sap1_mk2_custom:AT28C16
- added U47: 74LS161, symbol 74xx:74LS161
- added U48: 74LS138, symbol 74xx:74LS138
- added U49: 74LS00, symbol 74xx:74LS00
- added U50, U51: 74LS04, symbol 74xx:74LS04
Connections:
- new net: D64.1 (K), R83.2
- new net: D70.2 (A), U46.17 (D7), U51.1
- new net: D57.2 (A), R75.1
- new net: D67.1 (K), R86.2
- new net: D67.2 (A), U45.11 (D2), U50.13
- new net: U48.10 (O5), U49.5
- new net: U49.1, U49.2, U49.6
- new net: D68.2 (A), U45.10 (D1), U50.11
- new net: D66.2 (A), U45.13 (D3), U50.5
- new net: D65.2 (A), U45.14 (D4), U50.3
- new net: D63.2 (A), U45.16 (D6), U50.1
- new net: D56.2 (A), U45.6 (A2), U46.6 (A2), U47.12 (Q2), U48.3 (A2)
- new net: D55.2 (A), U45.7 (A1), U46.7 (A1), U47.13 (Q1), U48.2 (A1)
- new net: D54.2 (A), U45.8 (A0), U46.8 (A0), U47.14 (Q0), U48.1 (A0)
- new net: D69.2 (A), U45.9 (D0), U50.9
- new net: D76.2 (A), U46.10 (D1), U51.11
- new net: D75.2 (A), U46.11 (D2), U51.13
- new net: D72.2 (A), U46.15 (D5), U51.3
- new net: D77.2 (A), U46.9 (D0), U51.5
- new net: D60.2 (A), R78.1
- new net: D58.1 (K), U48.12 (O3)
- new net: D58.2 (A), R76.1
- new net: D65.1 (K), R84.2
- new net: D76.1 (K), R95.2
- new net: D75.1 (K), R94.2
- new net: D62.1 (K), R81.2
- new net: D61.1 (K), U48.15 (O0)
- new net: D61.2 (A), R79.1
- new net: D56.1 (K), R74.2
- new net: D69.1 (K), R88.2
- new net: D57.1 (K), U48.11 (O4)
- new net: D59.1 (K), U48.13 (O2)
- new net: D60.1 (K), U48.14 (O1)
- new net: D55.1 (K), R73.2
- new net: D72.1 (K), R91.2
- new net: R80.2, SW8.2, U49.10, U49.9
- new net: D71.1 (K), R90.2
- new net: D63.1 (K), R82.2
- new net: D74.1 (K), R93.2
- new net: D77.1 (K), R96.2
- new net: D66.1 (K), R85.2
- new net: D70.1 (K), R89.2
- new net: D73.1 (K), R92.2
- new net: D68.1 (K), R87.2
- new net: D59.2 (A), R77.1
- new net: U47.1 (~{MR}), U49.3
- new net: D54.1 (K), R72.2
- new net +5V: C48.1, C49.1, C50.1, C51.1, C52.2, C53.2, R75.2, R76.2, R77.2, R78.2, R79.2, SW8.1, U45.21 (~{WE}), U45.24 (VCC), U46.1 (A7), U46.21 (~{WE}), U46.24 (VCC), U47.10 (CET), U47.16 (VCC), U47.7 (CEP), U47.9 (~{PE}), U48.16 (VCC), U48.6 (E3), U49.14 (VCC), U50.14 (VCC)
- new net CE: D74.2 (A), U46.13 (D3)
- new net CF: U45.23 (A8), U46.23 (A8)
- new net CLR: U49.11
- new net GND: C48.2, C49.2, C50.2, C51.2, C52.1, C53.1, R72.1, R73.1, R74.1, R80.1, R81.1, R82.1, R83.1, R84.1, R85.1, R86.1, R87.1, R88.1, R89.1, R90.1, R91.1, R92.1, R93.1, R94.1, R95.1, R96.1, U45.1 (A7), U45.12 (GND), U45.18 (~{CE}), U45.19 (A10), U45.20 (~{OE}), U46.12 (GND), U46.18 (~{CE}), U46.19 (A10), U46.20 (~{OE}), U47.8 (GND), U48.4 (E1), U48.5 (E2), U48.8 (GND), U49.7 (GND), U50.7 (GND)
- new net HLT: D62.2 (A), U45.17 (D7)
- new net IR_4: U45.5 (A3), U46.5 (A3)
- new net IR_5: U45.4 (A4), U46.4 (A4)
- new net IR_6: U45.3 (A5), U46.3 (A5)
- new net IR_7: U45.2 (A6), U46.2 (A6)
- new net OI: D73.2 (A), U46.14 (D4)
- new net RI: D64.2 (A), U45.15 (D5)
- new net SU: D71.2 (A), U46.16 (D6)
- new net ZF: U45.22 (A9), U46.22 (A9)
- new net ~{AI}: U50.10
- new net ~{AO}: U50.8
- new net ~{BI}: U51.4
- new net ~{CLK}: U47.2 (CP)
- new net ~{CLR}: U49.12, U49.13, U49.4, U49.8
- new net ~{CO}: U51.12
- new net ~{EO}: U51.2
- new net ~{FI}: U51.6
- new net ~{II}: U50.12
- new net ~{IO}: U50.6
- new net ~{J}: U51.10
- new net ~{MI}: U50.2
- new net ~{RO}: U50.4
- no-connect marks 0 -> 10
Other:
- title: (none) -> Control Logic

Commit message: assigned footprints + finished root schematic
Parts:
- C48, C49, C50, C51, C52, C53: footprint (none) -> Capacitor_THT:C_Disc_D5.0mm_W2.5mm_P2.50mm
- D54, D55, D56, D57, D58, D59, D60, D61, D62, D63, D64, D65, D66, D67, D68, D69, D70, D71, D72, D73, D74, D75, D76, D77: footprint (none) -> LED_THT:LED_D3.0mm
- R72, R73, R74, R75, R76, R77, R78, R79, R80, R81, R82, R83, R84, R85, R86, R87, R88, R89, R90, R91, R92, R93, R94, R95, R96: footprint (none) -> Resistor_THT:R_Axial_DIN0207_L6.3mm_D2.5mm_P10.16mm_Horizontal
- SW8: footprint (none) -> Button_Switch_THT:SW_PUSH-12mm
- U47, U48: footprint (none) -> Package_DIP:DIP-16_W7.62mm
- U49, U50, U51: footprint (none) -> Package_DIP:DIP-14_W7.62mm
